File: HW6/ME433-2021/ME433-2021-1.brd (EAGLE design)
At the start: 160 x 100 mm, 56 parts, among them J1 B, J2 A, J3 str, J4 href, J5 pwdn

Commit message: submissions
Parts:
- R2: value 330 -> 10k
- moved J4 135.6 mm to (41.9, 12.7)
- moved J5 126.7 mm to (41.9, 25.4)
- moved J3 123.7 mm to (49.5, 27.9)
- moved U$10 84.0 mm to (142.2, 69.8), turned to 270 degrees
- moved U$6 82.1 mm to (47.0, 90.2), turned to 0 degrees
- moved C1 81.3 mm to (82.5, 82.5), turned to 270 degrees
- moved R2 80.5 mm to (34.3, 91.4), turned to 270 degrees
- moved J15 77.7 mm to (139.7, 108.0)
- moved LED1 76.7 mm to (15.2, 88.9)
- moved U$5 74.5 mm to (53.3, 76.2), turned to 0 degrees
- moved J14 72.0 mm to (143.5, 108.0)
- moved U$8 70.1 mm to (24.1, 34.3)
- moved J2 69.3 mm to (74.9, 113.0), turned to 90 degrees
- moved R1 68.9 mm to (24.1, 85.1)
- moved J13 66.5 mm to (147.3, 108.0)
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Connections:
- removed net N$5: R6.1, U$10.12
- removed net N$6: R7.1, U$10.13
- removed net N$8: U$9.7
- net +5V: no longer U$7.P$4
- net ADIR: now also U$12.P$9
- net APWM: now also U$12.P$10
- net B8: now also R6.1, U$10.12
- net B9: now also R7.1, U$10.13
- net BDIR: now also U$12.P$11
- net BPWM: now also U$12.P$12
- net D1: now also U$9.7
- net RCK: now also U$9.14
- net RRST: no longer U$9.14
Routing:
- net +3V3: track 0.00 -> 560.1 mm, vias 0 -> 1
- net VIN: track 0.00 -> 254.1 mm
- net B15: track 0.00 -> 138.6 mm, vias 0 -> 4
- net B0-PGD-D4: track 0.00 -> 127.9 mm
- net B13: track 0.00 -> 124.4 mm, vias 0 -> 3
- net B7: track 0.00 -> 121.5 mm, vias 0 -> 2
- net D6: track 0.00 -> 96.4 mm, vias 0 -> 3
- net D0: track 0.00 -> 95.3 mm, vias 0 -> 3
- net B6: track 0.00 -> 92.5 mm
- net B14: track 0.00 -> 91.5 mm, vias 0 -> 2
- net D2: track 0.00 -> 88.3 mm, vias 0 -> 5
- net B12: track 0.00 -> 87.3 mm, vias 0 -> 2
- net BPWM: track 0.00 -> 85.6 mm
- net B1-PGC-D5: track 0.00 -> 81.9 mm
- net D1: track 0.00 -> 80.5 mm, vias 0 -> 1
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- added copper zone on layer 16, net GND
Other:
- board size 160 x 100 mm -> 160 x 160 mm
- board text added: "Cassius Clay"
- board text added: "Motor A"
- board text added: "Motor B"
