File: HW6/ME433-2021/ME433-2021-1.sch (EAGLE design)
At the start: 56 parts, among them J1 B, J2 A, J3 str, J4 href, J5 pwdn

Commit message: submissions
Parts:
- R2: value 330 -> 10k
Connections:
- removed net N$5: R6.1, U$10.12.SCK
- removed net N$6: R7.1, U$10.13.SDA
- removed net N$8: U$9.7.D1
- net +5V: no longer U$7.4.5V
- net ADIR: now also U$12.9.ADIR
- net APWM: now also U$12.10.APWM
- net B8: now also R6.1, U$10.12.SCK
- net B9: now also R7.1, U$10.13.SDA
- net BDIR: now also U$12.11.BDIR
- net BPWM: now also U$12.12.BPWM
- net D1: now also U$9.7.D1
- net RCK: now also U$9.14.RCK
- net RRST: no longer U$9.14.RCK
Changed lines of the file:
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@@
 <part name="U$5" library="ME433-2021" deviceset="SNAP" device=""/>
 <part name="U$6" library="ME433-2021" deviceset="PUSH" device="" value="RESET"/>
-<part name="R2" library="ME433-2021" deviceset="R-US_" device="0207/10" package3d_urn="urn:adsk.eagle:package:23491/2" value="330"/>
+<part name="R2" library="ME433-2021" deviceset="R-US_" device="0207/10" package3d_urn="urn:adsk.eagle:package:23491/2" value="10k"/>
 <part name="C1" library="ME433-2021" deviceset="C-US" device="025-030X050" package3d_urn="urn:adsk.eagle:package:23631/1" value="0.1 uF"/>
 <part name="C2" library="ME433-2021" deviceset="C-US" device="025-030X050" package3d_urn="urn:adsk.eagle:package:23631/1" value="0.1 uF"/>
@@
 <part name="U$7" library="ME433-2021" deviceset="ADACP2104" device=""/>
 <part name="GND11" library="ME433-2021" deviceset="GND" device=""/>
-<part name="P+5" library="ME433-2021" deviceset="+5V" device=""/>
 <part name="U$8" library="ME433-2021" deviceset="ST7789" device=""/>
 <part name="GND12" library="ME433-2021" deviceset="GND" device=""/>
@@
 <attribute name="VALUE" x="114.3" y="101.6" size="1.778" layer="96"/>
 </instance>
-<instance part="P+5" gate="1" x="116.84" y="119.38" smashed="yes">
-<attribute name="VALUE" x="114.3" y="114.3" size="1.778" layer="96" rot="R90"/>
-</instance>
 <instance part="U$8" gate="G$1" x="175.26" y="119.38" smashed="yes">
 <attribute name="NAME" x="182.88" y="127" size="1.27" layer="94"/>
@@
 <wire x1="38.1" y1="104.14" x2="50.8" y2="104.14" width="0.1524" layer="91"/>
 </segment>
-<segment>
-<pinref part="P+5" gate="1" pin="+5V"/>
-<pinref part="U$7" gate="G$1" pin="4.5V"/>
-<wire x1="116.84" y1="116.84" x2="121.92" y2="116.84" width="0.1524" layer="91"/>
-</segment>
 </net>
 <net name="V+" class="0">
@@
 <label x="236.22" y="10.16" size="1.778" layer="95"/>
 </segment>
-<segment>
-<pinref part="U$9" gate="G$1" pin="14.RCK"/>
-<wire x1="223.52" y1="20.32" x2="236.22" y2="20.32" width="0.1524" layer="91"/>
-<label x="236.22" y="20.32" size="1.778" layer="95"/>
-</segment>
 </net>
 <net name="D0" class="0">
@@
 <label x="66.04" y="60.96" size="1.778" layer="95"/>
 </segment>
+<segment>
+<pinref part="U$9" gate="G$1" pin="7.D1"/>
+<wire x1="187.96" y1="30.48" x2="180.34" y2="30.48" width="0.1524" layer="91"/>
+<label x="180.34" y="30.48" size="1.778" layer="95"/>
+</segment>
 </net>
 <net name="D6" class="0">
@@
 <wire x1="78.74" y1="15.24" x2="66.04" y2="15.24" width="0.1524" layer="91"/>
 <label x="66.04" y="15.24" size="1.778" layer="95"/>
+</segment>
+<segment>
+<pinref part="U$9" gate="G$1" pin="14.RCK"/>
+<wire x1="223.52" y1="20.32" x2="238.76" y2="20.32" width="0.1524" layer="91"/>
+<label x="238.76" y="20.32" size="1.778" layer="95"/>
 </segment>
 </net>
@@
 <label x="129.54" y="15.24" size="1.778" layer="95"/>
 </segment>
+<segment>
+<pinref part="R6" gate="G$1" pin="1"/>
+<wire x1="190.5" y1="101.6" x2="190.5" y2="99.06" width="0.1524" layer="91"/>
+<wire x1="190.5" y1="99.06" x2="210.82" y2="99.06" width="0.1524" layer="91"/>
+<wire x1="210.82" y1="99.06" x2="210.82" y2="101.6" width="0.1524" layer="91"/>
+<pinref part="U$10" gate="G$1" pin="12.SCK"/>
+<wire x1="210.82" y1="101.6" x2="213.36" y2="101.6" width="0.1524" layer="91"/>
+<label x="210.82" y="101.6" size="1.778" layer="95"/>
+</segment>
 </net>
 <net name="B9" class="0">
@@
 <label x="124.46" y="20.32" size="1.778" layer="95"/>
 </segment>
+<segment>
+<pinref part="R7" gate="G$1" pin="1"/>
+<wire x1="182.88" y1="93.98" x2="213.36" y2="93.98" width="0.1524" layer="91"/>
+<pinref part="U$10" gate="G$1" pin="13.SDA"/>
+<wire x1="213.36" y1="93.98" x2="213.36" y2="96.52" width="0.1524" layer="91"/>
+<label x="208.28" y="93.98" size="1.778" layer="95"/>
+</segment>
 </net>
 <net name="D2" class="0">
@@
 <wire x1="223.52" y1="35.56" x2="236.22" y2="35.56" width="0.1524" layer="91"/>
 <label x="236.22" y="35.56" size="1.778" layer="95"/>
-</segment>
-</net>
-<net name="N$8" class="0">
-<segment>
-<pinref part="U$9" gate="G$1" pin="7.D1"/>
-<wire x1="187.96" y1="30.48" x2="180.34" y2="30.48" width="0.1524" layer="91"/>
-<label x="180.34" y="30.48" size="1.778" layer="95"/>
 </segment>
 </net>
@@
 </segment>
 </net>
-<net name="N$5" class="0">
-<segment>
-<pinref part="R6" gate="G$1" pin="1"/>
-<wire x1="190.5" y1="101.6" x2="190.5" y2="99.06" width="0.1524" layer="91"/>
-<wire x1="190.5" y1="99.06" x2="210.82" y2="99.06" width="0.1524" layer="91"/>
-<wire x1="210.82" y1="99.06" x2="210.82" y2="101.6" width="0.1524" layer="91"/>
-<pinref part="U$10" gate="G$1" pin="12.SCK"/>
-<wire x1="210.82" y1="101.6" x2="213.36" y2="101.6" width="0.1524" layer="91"/>
-</segment>
-</net>
-<net name="N$6" class="0">
-<segment>
-<pinref part="R7" gate="G$1" pin="1"/>
-<wire x1="182.88" y1="93.98" x2="213.36" y2="93.98" width="0.1524" layer="91"/>
-<pinref part="U$10" gate="G$1" pin="13.SDA"/>
-<wire x1="213.36" y1="93.98" x2="213.36" y2="96.52" width="0.1524" layer="91"/>
-</segment>
-</net>
 <net name="BPWM" class="0">
 <segment>
@@
 </segment>
 <segment>
-<wire x1="342.9" y1="132.08" x2="358.14" y2="132.08" width="0.1524" layer="91"/>
-<label x="358.14" y="132.08" size="1.778" layer="95"/>
+<pinref part="U$12" gate="G$1" pin="12.BPWM"/>
+<wire x1="342.9" y1="132.08" x2="365.76" y2="132.08" width="0.1524" layer="91"/>
+<label x="365.76" y="132.08" size="1.778" layer="95"/>
 </segment>
 </net>
@@
 </segment>
 <segment>
-<wire x1="342.9" y1="127" x2="358.14" y2="127" width="0.1524" layer="91"/>
-<label x="358.14" y="127" size="1.778" layer="95"/>
+<pinref part="U$12" gate="G$1" pin="11.BDIR"/>
+<wire x1="342.9" y1="127" x2="365.76" y2="127" width="0.1524" layer="91"/>
+<label x="365.76" y="127" size="1.778" layer="95"/>
 </segment>
 </net>
@@
 </segment>
 <segment>
-<wire x1="342.9" y1="121.92" x2="358.14" y2="121.92" width="0.1524" layer="91"/>
-<label x="358.14" y="121.92" size="1.778" layer="95"/>
+<pinref part="U$12" gate="G$1" pin="10.APWM"/>
+<wire x1="342.9" y1="121.92" x2="365.76" y2="121.92" width="0.1524" layer="91"/>
+<label x="365.76" y="121.92" size="1.778" layer="95"/>
 </segment>
 </net>
@@
 </segment>
 <segment>
-<wire x1="342.9" y1="116.84" x2="360.68" y2="116.84" width="0.1524" layer="91"/>
-<label x="360.68" y="116.84" size="1.778" layer="95"/>
-</segment>
-</net>
+<pinref part="U$12" gate="G$1" pin="9.ADIR"/>
+<wire x1="342.9" y1="116.84" x2="365.76" y2="116.84" width="0.1524" layer="91"/>
+<label x="365.76" y="116.84" size="1.778" layer="95"/>
+</segment>
+</net>
